File: shield/shield.sch (EAGLE design)
At the start: 27 parts, among them T2 2N2222, T5 2N2222, T6 2N2222, T9 2N2222

Commit message: Add files via upload
Parts:
- removed T2: 2N2222, adafruit:2N2222
- added T4: 2N2222, adafruit:2N2222
- J1, J10, J2, J3, J4, J7, J8, J9, LCD2, R1, R10, R2, R3, R4, R5, R6, R7, R8, R9, S1, S2, S3, T5, T6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: OC_FARNELL (none) -> unknown
- renumbered J6 to J7
Connections:
- removed net N$3: J7.2, T2.C
- new net N$25: J7.2, T4.C
- net GND: now also T4.E; no longer T2.E
- net N$26: now also T4.B; no longer T2.B
Other:
- moved on the sheet: LCD2
