File: shield/shield.brd (EAGLE design)
At the start: 100 x 80 mm, 27 parts, among them T2 2N2222, T5 2N2222, T6 2N2222, T9 2N2222

Commit message: Add files via upload
Parts:
- removed J6: (no value), con-amp:10X02MTA
- removed T2: 2N2222, adafruit:TO92-EBC-OVAL
- added J7: (no value), con-amp:10X02MTA
- added T4: 2N2222, adafruit:TO92-EBC-OVAL
- moved J2 24.1 mm to (39.4, 76.2), turned to 0 degrees
- moved J4 22.9 mm to (14.0, 76.2), turned to 0 degrees
- moved R2 19.7 mm to (76.2, 58.4)
- moved T6 17.8 mm to (91.4, 43.2)
- moved R3 16.1 mm to (76.2, 49.5)
- moved T9 15.3 mm to (91.4, 33.0)
- moved T5 15.3 mm to (91.4, 50.8)
- moved LCD2 14.0 mm to (43.2, 43.2)
- moved R4 13.7 mm to (76.2, 41.9)
- moved R5 9.16 mm to (76.2, 31.8)
- moved R7 8.98 mm to (17.8, 38.1), turned to 0 degrees
- moved R8 8.98 mm to (17.8, 43.2), turned to 0 degrees
- moved R9 8.98 mm to (17.8, 48.3), turned to 0 degrees
- moved R6 7.73 mm to (17.8, 31.8), turned to 0 degrees
- moved R1 7.62 mm to (40.6, 47.0)
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Connections:
- removed net N$3: J6.2, T2.C
- new net N$25: J7.2, T4.C
- net GND: now also T4.E; no longer T2.E
- net N$26: now also T4.B; no longer T2.B
- net VDD: now also J7.1; no longer J6.1
Routing:
- net N$25: track 0.00 -> 64.3 mm
- net N$32: track 168.2 -> 107.5 mm
- net N$33: track 165.0 -> 112.9 mm
- net GND: track 264.8 -> 314.8 mm
- net N$3: track 45.3 -> 0.00 mm
- net N$17: track 47.5 -> 8.33 mm
- net N$16: track 44.3 -> 21.6 mm
- net N$18: track 47.7 -> 25.4 mm
- net N$27: track 102.9 -> 123.6 mm, vias 1 -> 2
- net N$31: track 58.1 -> 38.4 mm
- net N$12: track 99.0 -> 116.2 mm, vias 0 -> 1
- net N$22: track 44.1 -> 59.2 mm
- net N$30: track 60.9 -> 46.4 mm
- net N$15: track 52.1 -> 42.4 mm
- net N$11: track 30.9 -> 22.3 mm
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